Commit message: update:已经支持场景中N个不同机械臂的加载,并预配置初始位置

File: src/robots_orchestra/scene/urdf/fanuc_crx10ia.urdf (robot description, URDF)
Before this commit: robot fanuc_crx10ia, 9 links, 8 joints
Links:
- link base_link: geometry collision mesh filename=meshes/fanuc_crx10ia/convex/base_link.ply; visual mesh filename=meshes/fanuc_crx10ia/visual/base_link.ply
- link link_1: geometry collision mesh filename=meshes/fanuc_crx10ia/convex/link_1.ply; visual mesh filename=meshes/fanuc_crx10ia/visual/link_1.ply
- link link_2: geometry collision mesh filename=meshes/fanuc_crx10ia/convex/link_2.ply; visual mesh filename=meshes/fanuc_crx10ia/visual/link_2.ply
- link link_3: geometry collision mesh filename=meshes/fanuc_crx10ia/convex/link_3.ply; visual mesh filename=meshes/fanuc_crx10ia/visual/link_3.ply
- link link_4: geometry collision mesh filename=meshes/fanuc_crx10ia/convex/link_4.ply; visual mesh filename=meshes/fanuc_crx10ia/visual/link_4.ply
- link link_5: geometry collision mesh filename=meshes/fanuc_crx10ia/convex/link_5.ply; visual mesh filename=meshes/fanuc_crx10ia/visual/link_5.ply
- link link_6: geometry collision mesh filename=meshes/fanuc_crx10ia/convex/link_6.ply; visual mesh filename=meshes/fanuc_crx10ia/visual/link_6.ply
