Commit message: update:初步完成了场景中碰撞物体的加载, 完善了目前的地安门框架

File: src/robots_orchestra/scene/urdf/abb_irb6700_150_320.urdf (robot description, URDF)
Before this commit: robot abb_irb6700_150_320, 7 links, 6 joints
Links:
- added link tool0
Joints:
- added joint tool0_joint: type fixed, parent link_6, child tool0, origin xyz=0 0 0 rpy=0 1.5707963267948966 0
