Commit message: update:初步完成了双击的搭建, franka机械臂的加入

File: src/robots_orchestra/scene/mobile/fanuc_car.urdf (robot description, URDF)
Before this commit: robot fanuc_car, 5 links, 4 joints
Joints:
- joint joint_1: axis 1 0 0 -> (none); limit lower=-20 upper=20 effort=100 velocity=10 -> (none); origin xyz=0 0 0 rpy=0 0 0 -> xyz=-0.234969 -0.493283 0.497258 rpy=0 0 0; type prismatic -> fixed
- joint joint_2: axis 0 1 0 -> (none); limit lower=-20 upper=20 effort=100 velocity=10 -> (none); type prismatic -> fixed
- joint joint_3: axis 0 0 1 -> (none); limit lower=-6.2832 upper=6.2832 effort=100 velocity=10 -> (none); type revolute -> fixed
- joint joint_4: parent move_y_link -> car_link
